File: kb_test/kb_test.kicad_pcb (KiCad board)
At the start: 2 copper layers, 323 x 117 mm, 171 parts, among them J1 Conn_01x04, SW1 SW_Push, SW10 SW_Push, SW11 SW_Push, SW12 SW_Push, SW13 SW_Push, SW14 SW_Push, SW15 SW_Push, SW16 SW_Push, SW17 SW_Push, SW18 SW_Push, SW19 SW_Push, SW2 SW_Push, SW20 SW_Push, SW21 SW_Push, SW22 SW_Push, SW23 SW_Push, SW24 SW_Push, SW25 SW_Push, SW26 SW_Push, SW27 SW_Push, SW28 SW_Push, SW29 SW_Push, SW3 SW_Push, SW30 SW_Push, SW31 SW_Push, SW32 SW_Push, SW33 SW_Push, SW34 SW_Push, SW35 SW_Push, SW36 SW_Push, SW37 SW_Push, SW38 SW_Push, SW39 SW_Push, SW4 SW_Push, SW40 SW_Push, SW41 SW_Push, SW42 SW_Push, SW43 SW_Push, SW44 SW_Push, SW45 SW_Push, SW46 SW_Push, SW47 SW_Push, SW48 SW_Push, SW49 SW_Push, SW5 SW_Push, SW50 SW_Push, SW51 SW_Push, SW52 SW_Push, SW53 SW_Push, SW54 SW_Push, SW55 SW_Push, SW56 SW_Push, SW57 SW_Push, SW58 SW_Push, SW59 SW_Push, SW6 SW_Push, SW60 SW_Push, SW61 SW_Push, SW62 SW_Push, SW63 SW_Push, SW64 SW_Push, SW65 SW_Push, SW66 SW_Push, SW67 SW_Push, SW68 SW_Push, SW69 SW_Push, SW7 SW_Push, SW70 SW_Push, SW71 SW_Push, SW72 SW_Push, SW73 SW_Push, SW74 SW_Push, SW75 SW_Push, SW76 SW_Push, SW77 SW_Push, SW78 SW_Push, SW79 SW_Push, SW8 SW_Push, SW80 SW_Push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

Commit message: Hardware as built; QMK firmware config OK
Parts:
- added H1: MountingHole, MountingHole:MountingHole_4.3mm_M4, F.Cu at (35.6, 155.6)
- added H2: MountingHole, MountingHole:MountingHole_4.3mm_M4, F.Cu at (35.6, 57.8)
- added H3: MountingHole, MountingHole:MountingHole_4.3mm_M4, F.Cu at (193.0, 155.6)
- added H4: MountingHole, MountingHole:MountingHole_4.3mm_M4, F.Cu at (327.0, 73.0)
- added H5: MountingHole, MountingHole:MountingHole_4.3mm_M4, F.Cu at (327.0, 114.9)
Routing:
- net COL13: track 0.00 -> 399.8 mm, vias 0 -> 1
- net ROW5: track 0.00 -> 399.7 mm, vias 0 -> 1
- net ROW4: track 0.00 -> 388.7 mm, vias 0 -> 1
- net COL9: track 0.00 -> 383.8 mm, vias 0 -> 1
- net COL8: track 0.00 -> 377.2 mm, vias 0 -> 2
- net COL14: track 0.00 -> 371.0 mm, vias 0 -> 1
- net ROW3: track 0.00 -> 370.4 mm, vias 0 -> 1
- net COL7: track 0.00 -> 366.8 mm, vias 0 -> 2
- net ROW2: track 0.00 -> 361.8 mm, vias 0 -> 1
- net COL12: track 0.00 -> 352.4 mm, vias 0 -> 3
- net COL6: track 0.00 -> 349.0 mm, vias 0 -> 3
- net COL11: track 0.00 -> 346.8 mm, vias 0 -> 2
- net COL15: track 0.00 -> 342.4 mm, vias 0 -> 1
- net ROW1: track 0.00 -> 339.9 mm, vias 0 -> 1
- net COL5: track 0.00 -> 330.5 mm, vias 0 -> 3
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- added copper zone on F.Cu, net GND
Other:
- board text added: "UPCO-84 Keyboard Rev 1.0 - 2025-03"
